File: kicad_files/XIAO ESP32C6/c6gdo.kicad_sch (KiCad schematic)
At the start: 10 parts, among them J1 250-1402, Q1 2N7002, Q2 AO3400A, U1 XIAO-ESP32-C6-SMD

Commit message: Add C5 support
Connections:
- net ESP_TX: now also U1.5 (GPIO22_D4_SDA); no longer U1.4 (GPIO21_D3)
Other:
- note added: "GPIO22 high turns Q2 on and pulls RED low (inverted UART TX). R1 holds Q2 off while the ESP32 is in reset or unpowered."
- note added: "NOTES 1. Firmware: ESPHome secplus_gdo (gdolib) with invert_uart = true; uart_tx_pin = GPIO22, uart_rx_pin = GPIO18. 2. Both FET stages invert the signal; the firmware's UART inversion restores the logic sense. 3. Q1's gate sees the RED line directly: use a part rated +/-20 V Vgs (do not substitute AO3400A, +/-12 V). 4. Ordering data: Manufacturer / MPN / Digi-Key PN symbol fields and c6gdo-bom.c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"
- note added: "Powered from the XIAO's own USB-C port (no board power input). ESP_TX = D4 / GPIO22 (uart_tx_pin) ESP_RX = D10 / GPIO18 (uart_rx_pin) Underside pads 24-33 (MTDI, MTDO, EN, GND, MTMS, MTCK, BOOT, 3V3, BAT, GND) are not soldered and are omitted from this symbol. The PCB footprint marks them with no-via keep-outs."
- note removed: "GPIO21 high turns Q2 on and pulls RED low (inverted UART TX). R1 holds Q2 off while the ESP32 is in reset or unpowered."
- note removed: "NOTES 1. Firmware: ESPHome secplus_gdo (gdolib) with invert_uart = true; uart_tx_pin = GPIO21, uart_rx_pin = GPIO18. 2. Both FET stages invert the signal; the firmware's UART inversion restores the logic sense. 3. Q1's gate sees the RED line directly: use a part rated +/-20 V Vgs (do not substitute AO3400A, +/-12 V). 4. Ordering data: Manufacturer / MPN / Digi-Key PN symbol fields and c6gdo-bom.c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"
- note removed: "Powered from the XIAO's own USB-C port (no board power input). ESP_TX = D3 / GPIO21 (uart_tx_pin) ESP_RX = D10 / GPIO18 (uart_rx_pin) Underside pads 24-33 (MTDI, MTDO, EN, GND, MTMS, MTCK, BOOT, 3V3, BAT, GND) are not soldered and are omitted from this symbol. The PCB footprint marks them with no-via keep-outs."

Commit message: D1 with better clamping voltage
Parts:
- D1: value CDSOD323-T15S -> PTVS15VS1UR; footprint c6gdo:D_SOD-323 -> c6gdo:Nexperia_CFP3_SOD-123W; symbol c6gdo:CDSOD323-T15S -> c6gdo:PTVS15VS1UR; Digi-Key PN CDSOD323-T15SCT-ND -> (none); DigiKey PN (none) -> 1727-5315-1-ND; MPN CDSOD323-T15S -> PTVS15VS1UR,115; Manufacturer Bourns Inc. -> Nexperia
- J1: Digi-Key PN 2946-250-1402-ND -> (none); DigiKey PN (none) -> 2946-250-1402-ND
- Q1: Digi-Key PN 2N7002NCT-ND -> (none); DigiKey PN (none) -> 2N7002NCT-ND
- Q2: Digi-Key PN 785-1000-1-ND -> (none); DigiKey PN (none) -> 785-1000-1-ND
- R1: Digi-Key PN P4.7KDACT-ND -> (none); DigiKey PN (none) -> P4.7KDACT-ND
- R2: Digi-Key PN P1.0KDACT-ND -> (none); DigiKey PN (none) -> P1.0KDACT-ND
- R3, R5: Digi-Key PN P123794CT-ND -> (none); DigiKey PN (none) -> P123794CT-ND
- R4: Digi-Key PN P100KDACT-ND -> (none); DigiKey PN (none) -> P100KDACT-ND
- U1: Digi-Key PN 1597-113991254-ND -> (none); DigiKey PN (none) -> 1597-113991254-ND
Other:
- note added: "NOTES 1. Firmware: ESPHome secplus_gdo (gdolib) with invert_uart = true; uart_tx_pin = GPIO22, uart_rx_pin = GPIO18. 2. Both FET stages invert the signal; the firmware's UART inversion restores the logic sense. 3. Q1's gate sees the RED line directly: use a part rated +/-20 V Vgs (do not substitute AO3400A, +/-12 V). 4. Ordering data: Manufacturer / MPN / DigiKey PN symbol fields and c6gdo-bom.cs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"
- note removed: "NOTES 1. Firmware: ESPHome secplus_gdo (gdolib) with invert_uart = true; uart_tx_pin = GPIO22, uart_rx_pin = GPIO18. 2. Both FET stages invert the signal; the firmware's UART inversion restores the logic sense. 3. Q1's gate sees the RED line directly: use a part rated +/-20 V Vgs (do not substitute AO3400A, +/-12 V). 4. Ordering data: Manufacturer / MPN / Digi-Key PN symbol fields and c6gdo-bom.c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"
Changed lines of the file:
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@@
 	(title_block
 		(title "XIAO ESP32-C6 Security+ 2.0 Garage Door Interface")
-		(date "2026-09-16")
-		(rev "1.0")
+		(date "2026-09-17")
+		(rev "1.1")
 		(company "MFLAGG")
 		(comment 1 "Derived from the rat-ratgdo D1 Mini - ESP32 board")
@@
 		)
 	)
-	(text "NOTES\n1. Firmware: ESPHome secplus_gdo (gdolib) with invert_uart = true; uart_tx_pin = GPIO22, uart_rx_pin = GPIO18.\n2. Both FET stages invert the signal; the firmware's UART inversion restores the logic sense.\n3. Q1's gate sees the RED line directly: use a part rated +/-20 V Vgs (do not substitute AO3400A, +/-12 V).\n4. Ordering data: Manufacturer / MPN / Digi-Key PN symbol fields and c6gdo-bom.csv."
+	(text "NOTES\n1. Firmware: ESPHome secplus_gdo (gdolib) with invert_uart = true; uart_tx_pin = GPIO22, uart_rx_pin = GPIO18.\n2. Both FET stages invert the signal; the firmware's UART inversion restores the logic sense.\n3. Q1's gate sees the RED line directly: use a part rated +/-20 V Vgs (do not substitute AO3400A, +/-12 V).\n4. Ordering data: Manufacturer / MPN / DigiKey PN symbol fields and c6gdo-bom.csv."
 		(exclude_from_sim no)
 		(at 22.86 157.48 0)
@@
 			)
 		)
-		(property "Digi-Key PN" "P123794CT-ND"
+		(property "DigiKey PN" "P123794CT-ND"
 			(at 138.43 127 0)
 			(hide yes)
@@
 			)
 		)
-		(property "Digi-Key PN" "P123794CT-ND"
+		(property "DigiKey PN" "P123794CT-ND"
 			(at 160.02 110.49 0)
 			(hide yes)
@@
 	)
 	(symbol
-		(lib_id "c6gdo:CDSOD323-T15S")
+		(lib_id "c6gdo:PTVS15VS1UR")
 		(at 220.98 62.23 270)
 		(unit 1)
@@
 			)
 		)
-		(property "Value" "CDSOD323-T15S"
+		(property "Value" "PTVS15VS1UR"
 			(at 223.52 63.5 90)
 			(show_name no)
@@
 			)
 		)
-		(property "Footprint" "c6gdo:D_SOD-323"
+		(property "Footprint" "c6gdo:Nexperia_CFP3_SOD-123W"
 			(at 220.98 62.23 0)
 			(hide yes)
@@
 			)
 		)
-		(property "Datasheet" "https://www.bourns.com/docs/product-datasheets/cdsod323-txxsc.pdf"
+		(property "Datasheet" "https://assets.nexperia.com/documents/data-sheet/PTVSXS1UR_SER.pdf"
 			(at 220.98 62.23 0)
 			(hide yes)
@@
 			)
 		)
-		(property "Description" "15V unidirectional TVS, SOD-323"
+		(property "Description" "15V 400W unidirectional TVS, SOD-123W"
 			(at 220.98 62.23 0)
 			(hide yes)
@@
 			)
 		)
-		(property "Manufacturer" "Bourns Inc."
+		(property "Manufacturer" "Nexperia"
 			(at 220.98 62.23 0)
 			(hide yes)
@@
 			)
 		)
-		(property "MPN" "CDSOD323-T15S"
+		(property "MPN" "PTVS15VS1UR,115"
 			(at 220.98 62.23 0)
 			(hide yes)
@@
 			)
 		)
-		(property "Digi-Key PN" "CDSOD323-T15SCT-ND"
+		(property "DigiKey PN" "1727-5315-1-ND"
 			(at 220.98 62.23 0)
 			(hide yes)
@@
 			)
 		)
-		(property "Digi-Key PN" "2946-250-1402-ND"
+		(property "DigiKey PN" "2946-250-1402-ND"
 			(at 261.62 58.42 0)
 			(hide yes)
@@
 			)
 		)
-		(property "Digi-Key PN" "1597-113991254-ND"
+		(property "DigiKey PN" "1597-113991254-ND"
 			(at 63.5 76.2 0)
 			(hide yes)
@@
 			)
 		)
-		(property "Digi-Key PN" "P4.7KDACT-ND"
+		(property "DigiKey PN" "P4.7KDACT-ND"
 			(at 129.54 64.77 0)
 			(hide yes)
@@
 			)
 		)
-		(property "Digi-Key PN" "P1.0KDACT-ND"
+		(property "DigiKey PN" "P1.0KDACT-ND"
 			(at 138.43 58.42 0)
 			(hide yes)
@@
 			)
 		)
-		(property "Digi-Key PN" "785-1000-1-ND"
+		(property "DigiKey PN" "785-1000-1-ND"
 			(at 152.4 58.42 0)
 			(hide yes)
@@
 			)
 		)
-		(property "Digi-Key PN" "2N7002NCT-ND"
+		(property "DigiKey PN" "2N7002NCT-ND"
 			(at 152.4 127 0)
 			(hide yes)
@@
 			)
 		)
-		(property "Digi-Key PN" "P100KDACT-ND"
+		(property "DigiKey PN" "P100KDACT-ND"
 			(at 243.84 62.23 0)
 			(hide yes)
